File: MCU Datalogger/_autosave-MCU Datalogger.kicad_pcb (KiCad board)
At the start: 2 copper layers, 50.8 x 30.5 mm, 31 parts, among them J1 Conn_01x04_Pin, J2 Conn_01x09_Pin, J3 Conn_01x04_Pin, J4 Conn_02x03_Odd_Even, U1 24LC1025, U2 DS1337S_, U3 24LC1025, U4 ATMEGA328P-AU, Y1 32.768KHz, Y2 16MHz

Commit message: main: updating main
Routing:
- net /SDA: track 71.1 -> 72.5 mm
- net /D9: track 20.3 -> 21.1 mm
- net Net-(D1-K): track 3.92 -> 4.58 mm
- net GND: track 208.5 -> 209.2 mm
- net /Vcc: track 240.9 -> 241.5 mm
