File: ESP32_demo_project/user_interface.kicad_sch (KiCad schematic)
At the start: 11 parts, among them J4 Conn_01x04_Pin, J5 Conn_01x05_Pin, Q2 BC817, Q3 BC817

Commit message: main: updating layout
Parts:
- S1, S2: footprint USLPT2819DT2TR:SW_USLPT2819DT2TR -> ESP32_project_Footprints:SW_USLPT2819DT2TR
Changed lines of the file:
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@@
 			)
 		)
-		(property "Footprint" "USLPT2819DT2TR:SW_USLPT2819DT2TR"
+		(property "Footprint" "ESP32_project_Footprints:SW_USLPT2819DT2TR"
 			(at 127 50.8 0)
 			(effects
@@
 			)
 		)
-		(property "Footprint" "USLPT2819DT2TR:SW_USLPT2819DT2TR"
+		(property "Footprint" "ESP32_project_Footprints:SW_USLPT2819DT2TR"
 			(at 171.45 54.61 0)
 			(effects
