File: ESP32_demo_project/ESP32_demo_project.kicad_sch (KiCad schematic)
At the start: 25 parts, among them J1 SS-52400-002, J2 B2B-PH-SM4-TB, U1 MCP73871

Commit message: main: closed out schematics
Parts:
- C1, C2, C5, C6: footprint (none) -> Capacitor_SMD:C_0805_2012Metric
- C3, C4: footprint (none) -> ESP32_project_Footprints:T491A
- F1: footprint FUSC3226X100N -> ESP32_project_Footprints:FUSC3226X100N
- LED1, LED2, LED3, LED4: footprint LEDC2012X120N -> ESP32_project_Footprints:LEDC2012X120N
- R1, R10, R2, R3, R4, R5, R6, R7, R8, R9: footprint (none) -> Resistor_SMD:R_0805_2012Metric
Connections:
- net USB_DN2 is gone; now on net USB_DN: J1.B7 (DN2)
- net USB_DP2 is gone; now on net USB_DP: J1.B6 (DP2)
- net +5V_VBUS: now also U1.4 (PROG2)
- net GND: now also U1.3 (SEL)
- net PWD_LED: now reaches LED4.1 (K), R10.1
- net USB_DN1 renamed USB_DN
- net USB_DP1 renamed USB_DP
Other:
- moved on the sheet: C2, C3, C4, C5, VR1

Commit message: main: updating layout
Parts:
- J1: footprint SS-52400-002:BELFUSE_SS-52400-002 -> ESP32_project_Footprints:BELFUSE_SS-52400-002
- J2: footprint B2B-PH-SM4-TB:JST_B2B-PH-SM4-TB -> ESP32_project_Footprints:JST_B2B-PH-SM4-TB
- VR1: footprint LM1117MPX-3.3:VREG_LM1117MPX-3.3 -> ESP32_project_Footprints:VREG_LM1117MPX-3.3
Changed lines of the file:
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@@
 			)
 		)
-		(property "Footprint" "SS-52400-002:BELFUSE_SS-52400-002"
+		(property "Footprint" "ESP32_project_Footprints:BELFUSE_SS-52400-002"
 			(at 63.5 62.23 0)
 			(effects
@@
 			)
 		)
-		(property "Footprint" "B2B-PH-SM4-TB:JST_B2B-PH-SM4-TB"
+		(property "Footprint" "ESP32_project_Footprints:JST_B2B-PH-SM4-TB"
 			(at 45.72 176.53 0)
 			(effects
@@
 			)
 		)
-		(property "Footprint" "LM1117MPX-3.3:VREG_LM1117MPX-3.3"
+		(property "Footprint" "ESP32_project_Footprints:VREG_LM1117MPX-3.3"
 			(at 64.77 130.81 0)
 			(effects
